File: PCB/Prototipo_2.0/BatteryGaulgue/BatteryGaulgue.kicad_sch (KiCad schematic)
At the start: 28 parts, among them J1 Screw_Terminal_01x03, J10 Conn_01x01_Pin, J2 Screw_Terminal_01x02, J3 Screw_Terminal_01x03, J4 Conn_01x01_Pin, J5 Conn_01x01_Pin, J6 Conn_01x01_Pin, J7 Screw_Terminal_01x02, J8 Conn_01x03_Pin, J9 Conn_01x01_Pin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

Commit message: Prototipos de la PCB del batteryGaulgue(falta rootear)
Parts:
- C1, C2, C3, C4, C5, C6: footprint Capacitor_THT:C_Rect_L7.0mm_W3.5mm_P5.00mm -> Capacitor_SMD:C_0805_2012Metric_Pad1.18x1.45mm_HandSolder
- R1, R2, R3, R4, R5, R7, R8: footprint Resistor_THT:R_Axial_DIN0207_L6.3mm_D2.5mm_P10.16mm_Horizontal -> Resistor_SMD:R_1206_3216Metric_Pad1.30x1.75mm_HandSolder
- U1: footprint TFG-BQ34Z1G:PW0014A_N -> BQ34Z100:SOP65P640X120-14N
Connections:
- no-connect marks 0 -> 1
Other:
- company: (none) -> UPM-Nizar El Azeouzi Amine
- title: (none) -> Battery Gaulge
- moved on the sheet: TH1
