File: PCB/Prototipo_2.0/BatteryGaulgue/BatteryGaulgue.kicad_pcb (KiCad board)
At the start: 2 copper layers, 68.5 x 38 mm, 32 parts, among them J1 Screw_Terminal_01x03, J10 Conn_01x01_Pin, J2 Screw_Terminal_01x02, J3 Screw_Terminal_01x03, J4 Conn_01x01_Pin, J5 Conn_01x01_Pin, J6 Conn_01x01_Pin, J7 Screw_Terminal_01x02, J8 Conn_01x03_Pin, J9 Conn_01x01_Pin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

Commit message: Placa PCB BatteryGaulgue terminada para fabricar
Parts:
- moved J4 14.0 mm to (130.0, 74.5)
- moved TH1 5.29 mm to (118.7, 96.0)
- moved C1 3.47 mm to (124.5, 89.2)
- moved C2 3.47 mm to (124.5, 82.2)
- moved R1 3.47 mm to (124.5, 85.8)
- moved R2 3.47 mm to (124.5, 79.2)
- moved C3 2.85 mm to (129.2, 83.8)
- moved Rshunt1 2.80 mm to (118.5, 82.2)
- moved J9 1.77 mm to (116.2, 91.2)
- moved J8 0.79 mm to (139.8, 64.2)
- moved J5 0.56 mm to (116.2, 75.0)
- moved C4 0.50 mm to (138.5, 76.5)
- moved M3 0.25 mm to (108.5, 95.2)
Routing:
- net Net-(J1-Pin_3): track 0.00 -> 89.5 mm, vias 0 -> 2
- net Net-(J3-Pin_1): track 0.00 -> 85.8 mm, vias 0 -> 3
- net Net-(J3-Pin_2): track 0.00 -> 84.0 mm
- net Net-(J3-Pin_3): track 0.00 -> 67.9 mm
- net Net-(J5-Pin_1): track 0.00 -> 54.2 mm, vias 0 -> 2
- net /REGIN: track 0.00 -> 50.3 mm, vias 0 -> 4
- net /REG25: track 0.00 -> 44.8 mm, vias 0 -> 2
- net Net-(J2-Pin_2): track 0.00 -> 41.5 mm, vias 0 -> 2
- net Net-(J2-Pin_1): track 0.00 -> 38.9 mm, vias 0 -> 2
- net Net-(U1-P6_TS): track 0.00 -> 32.6 mm
- net Net-(J6-Pin_1): track 0.00 -> 27.4 mm
- net Net-(J9-Pin_1): track 0.00 -> 26.8 mm
- net Net-(J7-Pin_1): track 0.00 -> 22.9 mm
- net Net-(J1-Pin_1): track 0.00 -> 15.3 mm
- net Net-(D1-K): track 0.00 -> 11.7 mm
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- added copper zone on B.Cu, net GND
- added copper zone on F.Cu, net GND
Other:
- board text added: "PCB_Prototype_BatteryGaulgue_ByPocheche"
