File: PCB/Prototipo_2.0/BatteryGaulgue/BatteryGaulgue.kicad_pcb (KiCad board)
At the start: 2 copper layers, 68.5 x 38 mm, 32 parts, among them J1 Screw_Terminal_01x03, J10 Conn_01x01_Pin, J2 Screw_Terminal_01x02, J3 Screw_Terminal_01x03, J4 Conn_01x01_Pin, J5 Conn_01x01_Pin, J6 Conn_01x01_Pin, J7 Screw_Terminal_01x02, J8 Conn_01x03_Pin, J9 Conn_01x01_Pin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

Commit message: .
Routing:
- net GND: track 1.96 -> 13.5 mm
Changed lines of the file:
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@@
 			(drillshape 0)
 			(scaleselection 1)
-			(outputdirectory "D:/GitHub/TFG-UPM/PCB/Prototipo_2.0/BatteryGaulgue/Fabricacion")
+			(outputdirectory "C:/Users/kille/Documents/GitHub/TFG-UPM/PCB/Prototipo_2.0/BatteryGaulgue/Fabricacion/")
 		)
 	)
@@
 		(layer "F.Cu")
 		(net 2)
+	)
+	(segment
+		(start 111.3275 85.5)
+		(end 118.3 85.5)
+		(width 2.5)
+		(layer "F.Cu")
+		(net 2)
+	)
+	(segment
+		(start 108.3275 82.5)
+		(end 111.3275 85.5)
+		(width 2.5)
+		(layer "F.Cu")
+		(net 2)
+	)
+	(segment
+		(start 118.3 85.5)
+		(end 118.5 85.3)
+		(width 2.5)
+		(layer "F.Cu")
+		(net 2)
