File: PCB/Prototipo_2.0/BatteryCharger_and_DCDCBuckBoost/converter.kicad_sch (KiCad schematic)
At the start: 1 part

Commit message: .
Other:
- company: (none) -> UPM-Nizar El Azeouzi Amine
- title: (none) -> Converter_DCDC_BuckBoost
- moved on the sheet: PS1
Changed lines of the file:
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@@
 	(generator_version "9.0")
 	(paper "A4")
+	(title_block
+		(title "Converter_DCDC_BuckBoost")
+		(date "2026-06-05")
+		(company "UPM-Nizar El Azeouzi Amine")
+	)
 	(symbol
 		(lib_id "LTC3115EFE-1_TRPBF:LTC3115EFE-1_TRPBF")
-		(at 135.89 71.12 0)
+		(at 142.24 78.74 0)
 		(unit 1)
 		(exclude_from_sim no)
@@
 		(fields_autoplaced yes)
 		(property "Reference" "PS1"
-			(at 135.89 45.72 0)
+			(at 142.24 53.34 0)
 			(effects
 				(font
@@
 		)
 		(property "Value" "LTC3115EFE-1_TRPBF"
-			(at 135.89 48.26 0)
+			(at 142.24 55.88 0)
 			(effects
 				(font
@@
 		)
 		(property "Footprint" "LTC3115EFE-1_TRPBF:CONV_LTC3115EFE-1_TRPBF"
-			(at 135.89 71.12 0)
+			(at 142.24 78.74 0)
 			(effects
 				(font
@@
 		)
 		(property "Datasheet" ""
-			(at 135.89 71.12 0)
+			(at 142.24 78.74 0)
 			(effects
 				(font
@@
 		)
 		(property "Description" ""
-			(at 135.89 71.12 0)
+			(at 142.24 78.74 0)
 			(effects
 				(font
@@
 		)
 		(property "MF" "Analog Devices"
-			(at 135.89 71.12 0)
+			(at 142.24 78.74 0)
 			(effects
 				(font
@@
 		)
 		(property "MAXIMUM_PACKAGE_HEIGHT" "1.2mm"
-			(at 135.89 71.12 0)
+			(at 142.24 78.74 0)
 			(effects
 				(font
@@
 		)
 		(property "Package" "TSSOP -20 Analog Devices"
-			(at 135.89 71.12 0)
+			(at 142.24 78.74 0)
 			(effects
 				(font
@@
 		)
 		(property "Price" "None"
-			(at 135.89 71.12 0)
+			(at 142.24 78.74 0)
 			(effects
 				(font
@@
 		)
 		(property "Check_prices" "https://www.snapeda.com/parts/LTC3115EFE-1%23TRPBF/Analog+Devices/view-part/?ref=eda"
-			(at 135.89 71.12 0)
+			(at 142.24 78.74 0)
 			(effects
 				(font
@@
 		)
 		(property "STANDARD" "Manufacturer Recommendations"
-			(at 135.89 71.12 0)
+			(at 142.24 78.74 0)
 			(effects
 				(font
@@
 		)
 		(property "PARTREV" "E"
-			(at 135.89 71.12 0)
+			(at 142.24 78.74 0)
 			(effects
 				(font
@@
 		)
 		(property "SnapEDA_Link" "https://www.snapeda.com/parts/LTC3115EFE-1%23TRPBF/Analog+Devices/view-part/?ref=snap"
-			(at 135.89 71.12 0)
+			(at 142.24 78.74 0)
 			(effects
 				(font
@@
 		)
 		(property "MP" "LTC3115EFE-1#TRPBF"
-			(at 135.89 71.12 0)
+			(at 142.24 78.74 0)
 			(effects
 				(font
@@
 		)
 		(property "Purchase-URL" "https://www.snapeda.com/api/url_track_click_mouser/?unipart_id=4338510&manufacturer=Analog Devices&part_name=LTC3115EFE-1#TRPBF&search_term=ltc3115efe-1#trpbf"
-			(at 135.89 71.12 0)
+			(at 142.24 78.74 0)
 			(effects
 				(font
@@
 		)
 		(property "Description_1" "40V, 2A Synchronous Buck-Boost DC/DC Converter"
-			(at 135.89 71.12 0)
+			(at 142.24 78.74 0)
 			(effects
 				(font
@@
 		)
 		(property "Availability" "In Stock"
-			(at 135.89 71.12 0)
+			(at 142.24 78.74 0)
 			(effects
 				(font
@@
 		)
 		(property "MANUFACTURER" "Analog Devices"
-			(at 135.89 71.12 0)
+			(at 142.24 78.74 0)
 			(effects
 				(font

Commit message: a
Parts:
- added C10: 10uF, Capacitor_SMD:C_0805_2012Metric_Pad1.18x1.45mm_HandSolder, symbol Device:C
- added C3, C5: 0.1uF, Capacitor_SMD:C_0805_2012Metric_Pad1.18x1.45mm_HandSolder, symbol Device:C
- added C6: 22uF, Capacitor_SMD:C_0805_2012Metric_Pad1.18x1.45mm_HandSolder, symbol Device:C
- added C7: 33pF, Capacitor_SMD:C_0805_2012Metric_Pad1.18x1.45mm_HandSolder, symbol Device:C
- added C8: 4.7uF, Capacitor_SMD:C_0805_2012Metric_Pad1.18x1.45mm_HandSolder, symbol Device:C
- added C9: 820pF, Capacitor_SMD:C_0805_2012Metric_Pad1.18x1.45mm_HandSolder, symbol Device:C
- added J6: Conn_01x03_Pin, Connector_PinHeader_2.54mm:PinHeader_1x03_P2.54mm_Vertical, symbol Connector:Conn_01x03_Pin
- added J7, J9: Conn_01x01_Pin, Connector_PinHeader_2.54mm:PinHeader_1x01_P2.54mm_Vertical, symbol Connector:Conn_01x01_Pin
- added L2: WE-PD_7332, WE-PD_7332:WE-PD_7332, symbol WE-PD_7332:WE-PD_7332
- added R10: 118k, Resistor_SMD:R_1206_3216Metric_Pad1.30x1.75mm_HandSolder, symbol Device:R
- added R11: 35.7k, Resistor_SMD:R_1206_3216Metric_Pad1.30x1.75mm_HandSolder, symbol Device:R
- added R5: 10k, Resistor_SMD:R_1206_3216Metric_Pad1.30x1.75mm_HandSolder, symbol Device:R
- added R6, R7, R9: 1M, Resistor_SMD:R_1206_3216Metric_Pad1.30x1.75mm_HandSolder, symbol Device:R
- added R8: 90.9k, Resistor_SMD:R_1206_3216Metric_Pad1.30x1.75mm_HandSolder, symbol Device:R
Connections:
- net PGND is gone; now on net GND: PS1.1 (PGND), PS1.10 (PGND), PS1.11 (PGND), PS1.20 (PGND), PS1.21 (PGND)
- net GND: now also C10.2, C6.2, C8.2, J6.3 (Pin_3), R10.1, R11.1, R8.2
- net at PS1.12 (VCC): now also PS1.14 (PVCC), PS1.19 (PWM/SYNC), C8.1
- net IN_DCDC: now reaches PS1.13 (VIN)
- net IN_DCDC: now also PS1.17 (PVIN), C10.1, J7.1 (Pin_1), R9.2
- net at PS1.15 (BST2): now also C5.2
- net at PS1.16 (BST1): now also C3.2
- net at PS1.18 (SW1): now also C3.1, L2.1
- net at PS1.2 (RUN): now also J6.2 (Pin_2)
- net at PS1.3 (SW2): now also C5.1, L2.2
- net Out_system: now reaches PS1.4 (PVOUT)
- net Out_system: now also C6.1, C7.2, J9.1 (Pin_1), R6.1
- net at PS1.7 (VC): now also R7.1
- net at PS1.8 (FB): now also C9.1, R5.2, R6.2, R8.1
- net at PS1.9 (RT): now also R11.2
- new net: C7.1, R5.1
- new net: C9.2, R7.2
- new net: J6.1 (Pin_1), R10.2, R9.1

Commit message: ...
Parts:
- C10, C3, C5, C6, C7, C8, C9: footprint Capacitor_SMD:C_0805_2012Metric_Pad1.18x1.45mm_HandSolder -> Capacitor_SMD:C_1206_3216Metric_Pad1.33x1.80mm_HandSolder
Changed lines of the file:
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@@
 			)
 		)
-		(property "Footprint" "Capacitor_SMD:C_0805_2012Metric_Pad1.18x1.45mm_HandSolder"
+		(property "Footprint" "Capacitor_SMD:C_1206_3216Metric_Pad1.33x1.80mm_HandSolder"
 			(at 84.7852 66.04 0)
 			(effects
@@
 			)
 		)
-		(property "Footprint" "Capacitor_SMD:C_0805_2012Metric_Pad1.18x1.45mm_HandSolder"
+		(property "Footprint" "Capacitor_SMD:C_1206_3216Metric_Pad1.33x1.80mm_HandSolder"
 			(at 103.8352 86.36 0)
 			(effects
@@
 			)
 		)
-		(property "Footprint" "Capacitor_SMD:C_0805_2012Metric_Pad1.18x1.45mm_HandSolder"
+		(property "Footprint" "Capacitor_SMD:C_1206_3216Metric_Pad1.33x1.80mm_HandSolder"
 			(at 182.88 72.0852 0)
 			(effects
@@
 			)
 		)
-		(property "Footprint" "Capacitor_SMD:C_0805_2012Metric_Pad1.18x1.45mm_HandSolder"
+		(property "Footprint" "Capacitor_SMD:C_1206_3216Metric_Pad1.33x1.80mm_HandSolder"
 			(at 187.96 60.6552 0)
 			(effects
@@
 			)
 		)
-		(property "Footprint" "Capacitor_SMD:C_0805_2012Metric_Pad1.18x1.45mm_HandSolder"
+		(property "Footprint" "Capacitor_SMD:C_1206_3216Metric_Pad1.33x1.80mm_HandSolder"
 			(at 184.15 96.2152 0)
 			(effects
@@
 			)
 		)
-		(property "Footprint" "Capacitor_SMD:C_0805_2012Metric_Pad1.18x1.45mm_HandSolder"
+		(property "Footprint" "Capacitor_SMD:C_1206_3216Metric_Pad1.33x1.80mm_HandSolder"
 			(at 182.5752 50.8 0)
 			(effects
@@
 			)
 		)
-		(property "Footprint" "Capacitor_SMD:C_0805_2012Metric_Pad1.18x1.45mm_HandSolder"
+		(property "Footprint" "Capacitor_SMD:C_1206_3216Metric_Pad1.33x1.80mm_HandSolder"
 			(at 203.5048 43.18 0)
 			(effects
