File: PCB/Prototipo_2.0/BatteryCharger_and_DCDCBuckBoost/Battery_and_DCDC.kicad_pcb (KiCad board)
At the start: 2 copper layers, 48 parts, among them J1 Screw_Terminal_01x02, J10 Screw_Terminal_01x02, J11 Conn_01x03_Pin, J12 PJ-002BH, J14 Conn_01x03_Pin, J15 Screw_Terminal_01x02, J16 Screw_Terminal_01x02, J2 Conn_01x01_Pin, J3 Conn_01x01_Pin, J4 Conn_01x01_Pin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

Commit message: ....
Parts:
- added M1: MountingHole_4.3mm_M4, MountingHole:MountingHole_4.3mm_M4, F.Cu at (140.0, 95.8)
- moved J5 73.7 mm to (192.5, 61.5)
- moved R4 63.0 mm to (194.8, 68.0)
- moved R3 62.9 mm to (194.8, 64.8), turned to 180 degrees
- moved J11 59.2 mm to (153.5, 85.0), turned to -90 degrees
- moved J12 56.7 mm to (150.1, 89.8), turned to -90 degrees
- moved R2 54.8 mm to (194.8, 72.0)
- moved J10 52.7 mm to (139.5, 83.0), turned to -90 degrees
- moved J3 47.3 mm to (185.2, 80.2)
- moved J4 41.2 mm to (158.5, 77.8)
- moved J1 40.2 mm to (193.0, 95.2), turned to 90 degrees
- moved J2 34.7 mm to (182.8, 93.2)
- moved D2 34.7 mm to (167.2, 80.8), turned to 180 degrees
- moved U1 33.8 mm to (162.3, 88.1)
- moved D1 33.2 mm to (150.8, 79.5), turned to 180 degrees
- moved J16 32.7 mm to (192.9, 83.8), turned to 90 degrees
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Routing:
- net /Battery_Charger/System_Load: track 36.9 -> 123.0 mm
- net /ConverterDC_DC/Out_system: track 0.00 -> 66.8 mm
- net Net-(J1-Pin_2): track 0.00 -> 56.4 mm, vias 0 -> 2
- net Net-(J1-Pin_1): track 0.00 -> 52.5 mm, vias 0 -> 2
- net Net-(U1-VFB): track 0.00 -> 47.6 mm, vias 0 -> 2
- net Net-(J14-Pin_1): track 0.00 -> 42.4 mm
- net Net-(J2-Pin_1): track 0.00 -> 33.5 mm
- net Net-(PS1-BST2): track 15.3 -> 42.0 mm, vias 1 -> 2
- net Net-(PS1-PVCC): track 3.41 -> 29.5 mm, vias 0 -> 3
- net Net-(D1-K): track 0.00 -> 23.3 mm
- net Net-(PS1-FB): track 0.00 -> 22.3 mm
- net Net-(PS1-SW2): track 0.00 -> 21.6 mm
- net Net-(D3-K): track 0.00 -> 21.0 mm, vias 0 -> 2
- net Net-(J8-Pin_2): track 0.00 -> 17.8 mm
- net Net-(D2-K): track 0.00 -> 17.3 mm
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- added copper zone on B.Cu, net GND
- added copper zone on F.Cu, net GND
Other:
- board outline added: 64.8 x 50.5 mm
- board text added: "PCB_Prototype_BatteryCharger_and_ConverterDCDC"
